File: Horn.kicad_sch (KiCad schematic)
At the start: 15 parts, among them U1 AP62300TWU, U2 AP2112K-3.3

Commit message: Added microcontroller
Parts:
- added C10, C9: 16pF, symbol Device:C
- added C11, C12, C13, C14, C17: 100nF, symbol Device:C
- added C15, C8: 1uF, symbol Device:C
- added C16: 10uF, symbol Device:C
- added D3: WS2812B, LED_SMD:LED_WS2812B-2020_PLCC4_2.0x2.0mm, symbol LED:WS2812B
- added J1: USB_C_Receptacle, Connector_USB:USB_C_Receptacle_Molex_105450-0101, symbol Connector:USB_C_Receptacle
- added JP1: SolderJumper, Jumper:SolderJumper-2_P1.3mm_Open_RoundedPad1.0x1.5mm, symbol Jumper:SolderJumper_2_Open
- added R3, R4, R5, R7, R8: 10k, symbol Device:R
- added R6: 0, symbol Device:R
- added SW1: Boot, Button_Switch_SMD:SW_SPST_Omron_B3FS-101xP, symbol Switch:SW_Push
- added SW2: Enable, Button_Switch_SMD:SW_SPST_Omron_B3FS-101xP, symbol Switch:SW_Push
- added Y1: Crystal, Crystal:Crystal_SMD_MicroCrystal_CC5V-T1A-2Pin_4.1x1.5mm, symbol Device:Crystal
Connections:
- net +12V: no longer C5.1, U2.1 (VIN), U2.3 (EN)
- net +3.3V: now also U3.11 (VDD3P3_RTC), U3.17 (VDD3P3_CPU), U3.2 (VDD3P3), U3.3 (VDD3P3), U3.31 (VDDA), U3.32 (VDDA), C11.1, C12.1, C13.1, C14.1, C15.1, C16.1, R3.1, R4.1, R5.1
- net +5V: now also C5.1, U2.1 (VIN), U2.3 (EN), JP1.2 (B); no longer C3.1, C4.1, L1.2, R1.1
- net GND: now also D1.3 (VSS), D2.3 (VSS), C10.2, C11.2, C12.2, C13.2, C14.2, C15.2, C16.2, C17.2, C8.2, C9.2, D3.3 (VSS), J1.A1 (GND), J1.A12 (GND), J1.B1 (GND), J1.B12 (GND), R7.2, R8.2, SW1.2, SW2.1
- net at D1.2 (DOUT): now also D2.4 (DIN)
- net RGB: now reaches D1.4 (DIN)
- net RGB: now also U3.16 (GPIO10)
- net at U3.14 (GPIO8): now also R4.2
- net at U3.15 (GPIO9): now also SW1.1
- net at U3.18 (VDD_SPI): now also C17.1
- net D-: now reaches U3.25 (GPIO18)
- net D-: now also J1.A7 (D-), J1.B7 (D-)
- net D+: now reaches U3.26 (GPIO19)
- net D+: now also J1.A6 (D+), J1.B6 (D+)
- net at U3.29 (XTAL_N): now also C10.1, Y1.2
- net at U3.30 (XTAL_P): now also R6.2
- net at U3.6 (GPIO2): now also R3.2
- net at U3.7 (CHIP_EN): now also C8.1, R5.2, SW2.2
- net at D2.2 (DOUT): now also D3.4 (DIN)
- new net: J1.B5 (CC2), R7.1
- new net: C3.1, C4.1, JP1.1 (A), L1.2, R1.1
- new net: C9.1, R6.1, Y1.1
- new net: J1.A4 (VBUS), J1.A9 (VBUS), J1.B4 (VBUS), J1.B9 (VBUS)
- new net: J1.A5 (CC1), R8.1
- no-connect marks 1 -> 3
Other:
- note added: "CONNECTORS"
- note added: "USB-C"
- moved on the sheet: C5, C6, C7, D1, D2, U2, U3

Commit message: Added Transceiver
Parts:
- removed J1: USB_C_Receptacle, Connector_USB:USB_C_Receptacle_Molex_105450-0101, symbol Connector:USB_C_Receptacle
- added C18, C20: 10uF, symbol Device:C
- added C19, C21: 1uF, symbol Device:C
- added J1, J3: RJ45_LED_Shielded, Connector_RJ:RJ45_Connfly_DS1128-09-S8xx-S_Horizontal, symbol Connector:RJ45_LED_Shielded
- added J2: USB_C_Receptacle_USB2.0, Connector_USB:USB_C_Receptacle_G-Switch_GT-USB-7010ASV, symbol Connector:USB_C_Receptacle_USB2.0
- added U4: TJA1042T-3, Package_SO:SOIC-8_3.9x4.9mm_P1.27mm, symbol Interface_CAN_LIN:TJA1042T-3
Connections:
- net +3.3V: now also C18.1, C19.1, U4.5 (VIO)
- net +5V: now also D1.1 (VDD), D2.1 (VDD), D3.1 (VDD), C20.1, C21.1, J2.A4 (VBUS), J2.A9 (VBUS), J2.B4 (VBUS), J2.B9 (VBUS), U4.3 (VCC)
- net D+: now also J2.A6 (D+), J2.B6 (D+)
- net D-: now also J2.A7 (D-), J2.B7 (D-)
- net GND: now also U3.33 (GND), C18.2, C19.2, C20.2, C21.2, J2.A1 (GND), J2.A12 (GND), J2.B1 (GND), J2.B12 (GND), U4.8 (STB)
- net at R7.1: now also J2.B5 (CC2)
- net at R8.1: now also J2.A5 (CC1)
- net CAN_RX: now reaches U3.10 (MTDI)
- net CAN_RX: now also U4.4 (RXD)
- net CAN_TX: now reaches U3.9 (MTMS)
- net CAN_TX: now also U4.1 (TXD)
- new net CANH: U4.7 (CANH)
- new net CANL: U4.6 (CANL)
- no-connect marks 3 -> 5
Other:
- moved on the sheet: C17, C5, C6, C7, D1, D2, D3, R7, R8, U2

Commit message: Chose component sizes
Parts:
- C1: footprint (none) -> Capacitor_SMD:C_0805_2012Metric
- C10, C11, C12, C13, C14, C15, C16, C17, C18, C19, C2, C20, C21, C3, C4, C5, C6, C7, C8, C9: footprint (none) -> Capacitor_SMD:C_0603_1608Metric
- L1: footprint (none) -> Inductor_SMD:L_Sunlord_SWPA4030S
- R1, R2, R3, R4, R5, R6, R7, R8: footprint (none) -> Resistor_SMD:R_0603_1608Metric
Changed lines of the file:
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@@
       (effects (font (size 1.27 1.27)) (justify left))
     )
-    (property "Footprint" "" (at 310.1848 39.37 0)
+    (property "Footprint" "Capacitor_SMD:C_0603_1608Metric" (at 310.1848 39.37 0)
       (effects (font (size 1.27 1.27)) hide)
     )
@@
       (effects (font (size 1.27 1.27)) (justify left))
     )
-    (property "Footprint" "" (at 319.7352 39.37 0)
+    (property "Footprint" "Capacitor_SMD:C_0603_1608Metric" (at 319.7352 39.37 0)
       (effects (font (size 1.27 1.27)) hide)
     )
@@
       (effects (font (size 1.27 1.27)) (justify left))
     )
-    (property "Footprint" "" (at 174.752 232.41 90)
+    (property "Footprint" "Resistor_SMD:R_0603_1608Metric" (at 174.752 232.41 90)
       (effects (font (size 1.27 1.27)) hide)
     )
@@
       (effects (font (size 1.27 1.27)) (justify left))
     )
-    (property "Footprint" "" (at 117.8052 189.23 0)
+    (property "Footprint" "Capacitor_SMD:C_0603_1608Metric" (at 117.8052 189.23 0)
       (effects (font (size 1.27 1.27)) hide)
     )
@@
       (effects (font (size 1.27 1.27)) (justify left))
     )
-    (property "Footprint" "" (at 106.68 206.0448 0)
+    (property "Footprint" "Capacitor_SMD:C_0603_1608Metric" (at 106.68 206.0448 0)
       (effects (font (size 1.27 1.27)) hide)
     )
@@
   )
   (symbol (lib_id "Device:C") (at 118.11 45.72 0) (unit 1)
-    (in_bom yes) (on_board yes) (dnp no)
+    (in_bom yes) (on_board yes) (dnp no) (fields_autoplaced)
     (property "Reference" "C4" (at 121.92 44.45 0)
       (effects (font (size 1.27 1.27)) (justify left))
@@
       (effects (font (size 1.27 1.27)) (justify left))
     )
-    (property "Footprint" "" (at 119.0752 49.53 0)
+    (property "Footprint" "Capacitor_SMD:C_0603_1608Metric" (at 119.0752 49.53 0)
       (effects (font (size 1.27 1.27)) hide)
     )
@@
       (effects (font (size 1.27 1.27)) (justify left))
     )
-    (property "Footprint" "" (at 83.5152 189.23 0)
+    (property "Footprint" "Capacitor_SMD:C_0603_1608Metric" (at 83.5152 189.23 0)
       (effects (font (size 1.27 1.27)) hide)
     )
@@
       (effects (font (size 1.27 1.27)) (justify left))
     )
-    (property "Footprint" "" (at 72.0852 189.23 0)
+    (property "Footprint" "Capacitor_SMD:C_0603_1608Metric" (at 72.0852 189.23 0)
       (effects (font (size 1.27 1.27)) hide)
     )
@@
       (effects (font (size 1.27 1.27)) (justify left))
     )
-    (property "Footprint" "" (at 37.592 212.09 90)
+    (property "Footprint" "Resistor_SMD:R_0603_1608Metric" (at 37.592 212.09 90)
       (effects (font (size 1.27 1.27)) hide)
     )
@@
       (effects (font (size 1.27 1.27)) (justify left))
     )
-    (property "Footprint" "" (at 211.7852 50.8 0)
+    (property "Footprint" "Capacitor_SMD:C_0603_1608Metric" (at 211.7852 50.8 0)
       (effects (font (size 1.27 1.27)) hide)
     )
@@
       (effects (font (size 1.27 1.27)) (justify left))
     )
-    (property "Footprint" "" (at 335.5848 39.37 0)
+    (property "Footprint" "Capacitor_SMD:C_0603_1608Metric" (at 335.5848 39.37 0)
       (effects (font (size 1.27 1.27)) hide)
     )
@@
       (effects (font (size 1.27 1.27)) (justify left))
     )
-    (property "Footprint" "" (at 88.392 45.72 90)
+    (property "Footprint" "Resistor_SMD:R_0603_1608Metric" (at 88.392 45.72 90)
       (effects (font (size 1.27 1.27)) hide)
     )
@@
       (effects (font (size 1.27 1.27)) (justify left))
     )
-    (property "Footprint" "" (at 40.9448 46.99 0)
+    (property "Footprint" "Capacitor_SMD:C_0805_2012Metric" (at 40.9448 46.99 0)
       (effects (font (size 1.27 1.27)) hide)
     )
@@
   )
   (symbol (lib_id "Device:C") (at 106.68 45.72 0) (unit 1)
-    (in_bom yes) (on_board yes) (dnp no)
+    (in_bom yes) (on_board yes) (dnp no) (fields_autoplaced)
     (property "Reference" "C3" (at 110.49 44.45 0)
       (effects (font (size 1.27 1.27)) (justify left))
@@
       (effects (font (size 1.27 1.27)) (justify left))
     )
-    (property "Footprint" "" (at 107.6452 49.53 0)
+    (property "Footprint" "Capacitor_SMD:C_0603_1608Metric" (at 107.6452 49.53 0)
       (effects (font (size 1.27 1.27)) hide)
     )
@@
       (effects (font (size 1.27 1.27)) (justify left))
     )
-    (property "Footprint" "" (at 45.212 233.68 90)
+    (property "Footprint" "Resistor_SMD:R_0603_1608Metric" (at 45.212 233.68 90)
       (effects (font (size 1.27 1.27)) hide)
     )
@@
       (effects (font (size 1.27 1.27)) (justify left))
     )
-    (property "Footprint" "" (at 88.392 55.88 90)
+    (property "Footprint" "Resistor_SMD:R_0603_1608Metric" (at 88.392 55.88 90)
       (effects (font (size 1.27 1.27)) hide)
     )
@@
       (effects (font (size 1.27 1.27)) (justify left))
     )
-    (property "Footprint" "" (at 345.1352 39.37 0)
+    (property "Footprint" "Capacitor_SMD:C_0603_1608Metric" (at 345.1352 39.37 0)
       (effects (font (size 1.27 1.27)) hide)
     )
@@
       (effects (font (size 1.27 1.27)) (justify left))
     )
-    (property "Footprint" "" (at 47.9552 248.92 0)
+    (property "Footprint" "Capacitor_SMD:C_0603_1608Metric" (at 47.9552 248.92 0)
       (effects (font (size 1.27 1.27)) hide)
     )
@@
       (effects (font (size 1.27 1.27)) (justify left))
     )
-    (property "Footprint" "" (at 94.9452 189.23 0)
+    (property "Footprint" "Capacitor_SMD:C_0603_1608Metric" (at 94.9452 189.23 0)
       (effects (font (size 1.27 1.27)) hide)
     )
@@
       (effects (font (size 1.27 1.27)) (justify left))
     )
-    (property "Footprint" "" (at 201.6252 50.8 0)
+    (property "Footprint" "Capacitor_SMD:C_0603_1608Metric" (at 201.6252 50.8 0)
       (effects (font (size 1.27 1.27)) hide)
     )
@@
       (effects (font (size 1.27 1.27)) (justify left))
     )
-    (property "Footprint" "" (at 106.3752 189.23 0)
+    (property "Footprint" "Capacitor_SMD:C_0603_1608Metric" (at 106.3752 189.23 0)
       (effects (font (size 1.27 1.27)) hide)
     )
@@
       (effects (font (size 1.27 1.27)) (justify left))
     )
-    (property "Footprint" "" (at 35.2552 209.55 0)
+    (property "Footprint" "Capacitor_SMD:C_0603_1608Metric" (at 35.2552 209.55 0)
       (effects (font (size 1.27 1.27)) hide)
     )
@@
       (effects (font (size 1.27 1.27)) (justify left))
     )
-    (property "Footprint" "" (at 117.602 232.41 90)
+    (property "Footprint" "Resistor_SMD:R_0603_1608Metric" (at 117.602 232.41 90)
       (effects (font (size 1.27 1.27)) hide)
     )
@@
       (effects (font (size 1.27 1.27)) (justify left))
     )
-    (property "Footprint" "" (at 171.1452 50.8 0)
+    (property "Footprint" "Capacitor_SMD:C_0603_1608Metric" (at 171.1452 50.8 0)
       (effects (font (size 1.27 1.27)) hide)
     )
@@
       (effects (font (size 1.27 1.27)))
     )
-    (property "Footprint" "" (at 83.82 41.91 0)
+    (property "Footprint" "Inductor_SMD:L_Sunlord_SWPA4030S" (at 83.82 41.91 0)
       (effects (font (size 1.27 1.27)) hide)
     )
@@
       (effects (font (size 1.27 1.27)) (justify left))
     )
-    (property "Footprint" "" (at 125.222 232.41 90)
+    (property "Footprint" "Resistor_SMD:R_0603_1608Metric" (at 125.222 232.41 90)
       (effects (font (size 1.27 1.27)) hide)
     )
@@
       (effects (font (size 1.27 1.27)) (justify left))
     )
-    (property "Footprint" "" (at 165.862 232.41 90)
+    (property "Footprint" "Resistor_SMD:R_0603_1608Metric" (at 165.862 232.41 90)
       (effects (font (size 1.27 1.27)) hide)
     )
@@
       (effects (font (size 1.27 1.27)) (justify left))
     )
-    (property "Footprint" "" (at 129.2352 189.23 0)
+    (property "Footprint" "Capacitor_SMD:C_0603_1608Metric" (at 129.2352 189.23 0)
       (effects (font (size 1.27 1.27)) hide)
     )
@@
   )
   (symbol (lib_id "Device:C") (at 74.93 36.83 90) (unit 1)
-    (in_bom yes) (on_board yes) (dnp no)
-    (property "Reference" "C2" (at 78.74 34.29 90)
-      (effects (font (size 1.27 1.27)) (justify left))
-    )
-    (property "Value" "100nF" (at 78.74 31.75 90)
-      (effects (font (size 1.27 1.27)) (justify left))
-    )
-    (property "Footprint" "" (at 78.74 35.8648 0)
+    (in_bom yes) (on_board yes) (dnp no) (fields_autoplaced)
+    (property "Reference" "C2" (at 74.93 29.21 90)
+      (effects (font (size 1.27 1.27)))
+    )
+    (property "Value" "100nF" (at 74.93 31.75 90)
+      (effects (font (size 1.27 1.27)))
+    )
+    (property "Footprint" "Capacitor_SMD:C_0603_1608Metric" (at 78.74 35.8648 0)
       (effects (font (size 1.27 1.27)) hide)
     )
@@
       (effects (font (size 1.27 1.27)) (justify left))
     )
-    (property "Footprint" "" (at 54.3052 209.55 0)
-      (effects (font (size 1.27 1.27)) hide)
-    )
+    (property "Footprint" "Capacitor_SMD:C_0603_1608Metric" (at 54.3052 209.55 0)
+      (effects (font (size 1.27 1.27)) hide)
+    )

Commit message: Started PCB
Parts:
- added J4: Screw_Terminal_01x02, TerminalBlock_MetzConnect:TerminalBlock_MetzConnect_Type011_RT05502HBWC_1x02_P5.00mm_Horizontal, symbol Connector:Screw_Terminal_01x02
- C3, C4, C7: footprint Capacitor_SMD:C_0603_1608Metric -> Capacitor_SMD:C_0805_2012Metric
Connections:
- net +12V: now also J4.1 (Pin_1)
- net +5V: now also J1.8, J3.8
- net CANH: now also J1.3, J3.3
- net CANL: now also J1.2, J3.2
- net GND: now also J1.1, J3.1, J4.2 (Pin_2)
- net at U1.2 (SW): now also C2.2, L1.1; no longer C2.1
- new net: C2.1, U1.6 (BST)
- no-connect marks 5 -> 13
Other:
- moved on the sheet: C2, C3, C4, J1, J3, JP1, L1, R1, R2
